Commit message: updated - sign camera.xacro

File: src/universal_robot/ur_description/urdf/camera.xacro (robot description, xacro)
@@ -9,5 +9,5 @@
         <parent link="wrist_3_link"/>
         <child link="camera_link_r"/>
-        <origin  xyz="0 0.023 0.02" rpy="0.0 0.0 0.0"/>
+        <origin  xyz="0 -0.023 0.02" rpy="0.0 0.0 0.0"/>
     </joint>
     <link name="camera_link_r">
